File: sega-gamegear-audio-original.kicad_sch (KiCad schematic)
At the start: 20 parts, among them CN1 CONN 2P, CN2 292161-6, IC1 TDA2822D, J1 PJ-307A

Commit message: update 3d models
Parts:
- C1, C2: footprint EEEFN1E101UP -> Sega GameGear Audio Board Original:C63D
- C3: footprint Sega GameGear Audio Board Original:EEEFT0J331AP -> Sega GameGear Audio Board Original:C63D
- C4, C6, C8, C9: footprint C0603 -> Sega GameGear Audio Board Original:C0603
- C5, C7: footprint EEEFK1C470P -> Sega GameGear Audio Board Original:C63D
Changed lines of the file:
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@@
       (effects (font (size 1.27 1.27)) (justify left))
     )
-    (property "Footprint" "EEEFN1E101UP" (at 113.03 83.82 0)
+    (property "Footprint" "Sega GameGear Audio Board Original:C63D" (at 113.03 83.82 0)
       (effects (font (size 1.27 1.27)) (justify left top) hide)
     )
@@
       (effects (font (size 1.27 1.27)) (justify left))
     )
-    (property "Footprint" "EEEFN1E101UP" (at 113.03 106.68 0)
+    (property "Footprint" "Sega GameGear Audio Board Original:C63D" (at 113.03 106.68 0)
       (effects (font (size 1.27 1.27)) (justify left top) hide)
     )
@@
       (effects (font (size 1.27 1.27)) (justify right))
     )
-    (property "Footprint" "C0603" (at 179.07 95.25 0)
+    (property "Footprint" "Sega GameGear Audio Board Original:C0603" (at 179.07 95.25 0)
       (effects (font (size 1.27 1.27)) (justify left top) hide)
     )
@@
       (effects (font (size 1.27 1.27)))
     )
-    (property "Footprint" "EEEFK1C470P" (at 158.75 83.82 0)
+    (property "Footprint" "Sega GameGear Audio Board Original:C63D" (at 158.75 83.82 0)
       (effects (font (size 1.27 1.27)) (justify left top) hide)
     )
@@
       (effects (font (size 1.27 1.27)) (justify right))
     )
-    (property "Footprint" "C0603" (at 212.09 72.39 0)
+    (property "Footprint" "Sega GameGear Audio Board Original:C0603" (at 212.09 72.39 0)
       (effects (font (size 1.27 1.27)) (justify left top) hide)
     )
@@
       (effects (font (size 1.27 1.27)) (justify right))
     )
-    (property "Footprint" "C0603" (at 179.07 120.65 0)
+    (property "Footprint" "Sega GameGear Audio Board Original:C0603" (at 179.07 120.65 0)
       (effects (font (size 1.27 1.27)) (justify left top) hide)
     )
@@
       (effects (font (size 1.27 1.27)) (justify left))
     )
-    (property "Footprint" "Sega GameGear Audio Board Original:EEEFT0J331AP" (at 143.51 48.26 0)
+    (property "Footprint" "Sega GameGear Audio Board Original:C63D" (at 143.51 48.26 0)
       (effects (font (size 1.27 1.27)) (justify left top) hide)
     )
@@
       (effects (font (size 1.27 1.27)))
     )
-    (property "Footprint" "EEEFK1C470P" (at 158.75 109.22 0)
+    (property "Footprint" "Sega GameGear Audio Board Original:C63D" (at 158.75 109.22 0)
       (effects (font (size 1.27 1.27)) (justify left top) hide)
     )
@@
       (effects (font (size 1.27 1.27)) (justify right))
     )
-    (property "Footprint" "C0603" (at 180.34 64.77 0)
-      (effects (font (size 1.27 1.27)) (justify left top) hide)
-    )
+    (property "Footprint" "Sega GameGear Audio Board Original:C0603" (at 180.34 64.77 0)
+      (effects (font (size 1.27 1.27)) (justify left top) hide)
+    )

Commit message: add vr1 footprint
Parts:
- removed RV1: evutv2b19a14, symbol evutv2b19a14:evutv2b19a14
- added VR1: EVUTV2B19A14, Sega GameGear Audio Board Original:EVUTV2B19A14, symbol EVUTV2B19A14:EVUTV2B19A14
Connections:
- net GND: now also VR1.5
- net at IC1.6 (+I2): now also VR1.4
- net at IC1.7 (+I1): now also VR1.2
- net at R1.2: now also VR1.1
- net at R2.2: now also VR1.3
Changed lines of the file:
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@@
-    )
-  )
-  (symbol (lib_id "evutv2b19a14:evutv2b19a14") (at 99.06 86.36 0) (unit 1)
-    (in_bom yes) (on_board yes) (dnp no)
-    (property "Reference" "RV1" (at 97.79 83.82 0)
-      (effects (font (size 1.27 1.27)))
-    )
-    (property "Value" "evutv2b19a14" (at 100.33 97.79 0)
-      (effects (font (size 1.27 1.27)))
-    )
-    (property "Footprint" "" (at 92.71 94.615 0)
-      (effects (font (size 1.27 1.27)) hide)
-    )
-    (property "Datasheet" "~" (at 92.71 94.615 0)
-      (effects (font (size 1.27 1.27)) hide)
-    )
-    (pin "1")
-    (pin "2")
-    (pin "3")
-    (pin "4")
-    (pin "5")
-    (instances
-      (project "sega-gamegear-audio-original"
-        (path "/bc4894cb-9ef9-4d80-9ba0-901cc46c914e"
-          (reference "RV1") (unit 1)
-        )
-      )
     )
   )
@@
         )
       )
+    )
+  )
+  (symbol (lib_id "EVUTV2B19A14:EVUTV2B19A14") (at 99.06 86.36 0) (unit 1)
+    (in_bom yes) (on_board yes) (dnp no) (fields_autoplaced)
+    (property "Reference" "VR1" (at 106.68 87.2491 0)
+      (effects (font (size 1.27 1.27)))
+    )
+    (property "Value" "EVUTV2B19A14" (at 106.68 89.7891 0)
+      (effects (font (size 1.27 1.27)))
+    )
+    (property "Footprint" "Sega GameGear Audio Board Original:EVUTV2B19A14" (at 91.44 107.95 0)
+      (effects (font (size 1.27 1.27)) hide)
+    )
+    (property "Datasheet" "~" (at 92.71 94.615 0)
+      (effects (font (size 1.27 1.27)) hide)
+    )
+    (pin "1")
+    (pin "2")
+    (pin "3")
+    (pin "4")
+    (pin "5")
+    (instances
+      (project "sega-gamegear-audio-original"
+        (path "/bc4894cb-9ef9-4d80-9ba0-901cc46c914e"
+          (reference "VR1") (unit 1)
+        )
+      )

Commit message: add board outline
Parts:
- J1: value PJ-307A -> CONN MINI JACK; Manufacturer_Part_Number (none) -> PJ-307A
Connections:
- net GND: no longer J1.12, J1.13, J1.14, J1.15, J1.7, J1.8, J1.9
Other:
- moved on the sheet: C1, C2, C3, C4, C5, C6, C7, C8, C9, CN1, CN2, IC1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

Commit message: add board settings for jlcpcb
Connections:
- net at IC1.5 (-I2): now also C2.1; no longer C1.1
- net at IC1.8 (-I1): now also C1.1; no longer C2.1
Changed lines of the file:
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@@
-    )
-  )
-  (symbol (lib_id "EEEFN1E101UP:EEEFN1E101UP") (at 113.03 90.17 270) (unit 1)
-    (in_bom yes) (on_board yes) (dnp no) (fields_autoplaced)
-    (property "Reference" "C2" (at 115.57 87.1982 90)
-      (effects (font (size 1.27 1.27)) (justify left))
-    )
-    (property "Value" "100uF" (at 115.57 89.7382 90)
-      (effects (font (size 1.27 1.27)) (justify left))
-    )
-    (property "Footprint" "Sega GameGear Audio Board Original:C63D" (at 109.22 83.82 0)
-      (effects (font (size 1.27 1.27)) (justify left top) hide)
-    )
-    (property "Datasheet" "http://industrial.panasonic.com/cdbs/www-data/pdf/RDE0000/RDE0000C1259.pdf" (at 105.41 53.34 0)
-      (effects (font (size 1.27 1.27)) (justify left top) hide)
-    )
-    (property "Height" "7.8" (at -283.16 99.06 0)
-      (effects (font (size 1.27 1.27)) (justify left top) hide)
-    )
-    (property "Manufacturer_Name" "Panasonic" (at -583.16 99.06 0)
-      (effects (font (size 1.27 1.27)) (justify left top) hide)
-    )
-    (property "Manufacturer_Part_Number" "EEEFN1E101UP" (at 115.57 92.2782 90)
-      (effects (font (size 1.27 1.27)) (justify left))
-    )
-    (pin "1")
-    (pin "2")
-    (instances
-      (project "sega-gamegear-audio-original"
-        (path "/bc4894cb-9ef9-4d80-9ba0-901cc46c914e"
-          (reference "C2") (unit 1)
-        )
-      )
-    )
-  )
-  (symbol (lib_id "EEEFN1E101UP:EEEFN1E101UP") (at 113.03 113.03 270) (unit 1)
-    (in_bom yes) (on_board yes) (dnp no) (fields_autoplaced)
-    (property "Reference" "C1" (at 115.57 110.0582 90)
-      (effects (font (size 1.27 1.27)) (justify left))
-    )
-    (property "Value" "100uF" (at 115.57 112.5982 90)
-      (effects (font (size 1.27 1.27)) (justify left))
-    )
-    (property "Footprint" "Sega GameGear Audio Board Original:C63D" (at 109.22 106.68 0)
-      (effects (font (size 1.27 1.27)) (justify left top) hide)
-    )
-    (property "Datasheet" "http://industrial.panasonic.com/cdbs/www-data/pdf/RDE0000/RDE0000C1259.pdf" (at 105.41 76.2 0)
-      (effects (font (size 1.27 1.27)) (justify left top) hide)
-    )
-    (property "Height" "7.8" (at -283.16 121.92 0)
-      (effects (font (size 1.27 1.27)) (justify left top) hide)
-    )
-    (property "Manufacturer_Name" "Panasonic" (at -583.16 121.92 0)
-      (effects (font (size 1.27 1.27)) (justify left top) hide)
-    )
-    (property "Manufacturer_Part_Number" "EEEFN1E101UP" (at 115.57 115.1382 90)
-      (effects (font (size 1.27 1.27)) (justify left))
-    )
-    (pin "1")
-    (pin "2")
-    (instances
-      (project "sega-gamegear-audio-original"
-        (path "/bc4894cb-9ef9-4d80-9ba0-901cc46c914e"
-          (reference "C1") (unit 1)
-        )
-      )
     )
   )
@@
     )
   )
+  (symbol (lib_id "EEEFN1E101UP:EEEFN1E101UP") (at 113.03 90.17 270) (unit 1)
+    (in_bom yes) (on_board yes) (dnp no) (fields_autoplaced)
+    (property "Reference" "C1" (at 115.57 87.1982 90)
+      (effects (font (size 1.27 1.27)) (justify left))
+    )
+    (property "Value" "100uF" (at 115.57 89.7382 90)
+      (effects (font (size 1.27 1.27)) (justify left))
+    )
+    (property "Footprint" "Sega GameGear Audio Board Original:C63D" (at 109.22 83.82 0)
+      (effects (font (size 1.27 1.27)) (justify left top) hide)
+    )
+    (property "Datasheet" "http://industrial.panasonic.com/cdbs/www-data/pdf/RDE0000/RDE0000C1259.pdf" (at 105.41 53.34 0)
+      (effects (font (size 1.27 1.27)) (justify left top) hide)
+    )
+    (property "Height" "7.8" (at -283.16 99.06 0)
+      (effects (font (size 1.27 1.27)) (justify left top) hide)
+    )
+    (property "Manufacturer_Name" "Panasonic" (at -583.16 99.06 0)
+      (effects (font (size 1.27 1.27)) (justify left top) hide)
+    )
+    (property "Manufacturer_Part_Number" "EEEFN1E101UP" (at 115.57 92.2782 90)
+      (effects (font (size 1.27 1.27)) (justify left))
+    )
+    (pin "1")
+    (pin "2")
+    (instances
+      (project "sega-gamegear-audio-original"
+        (path "/bc4894cb-9ef9-4d80-9ba0-901cc46c914e"
+          (reference "C1") (unit 1)
+        )
+      )
+    )
+  )
   (symbol (lib_id "RT0603BRD07100RL:RT0603BRD07100RL") (at 184.15 80.01 0) (unit 1)
     (in_bom yes) (on_board yes) (dnp no) (fields_autoplaced)
@@
         )
       )
+    )
+  )
+  (symbol (lib_id "EEEFN1E101UP:EEEFN1E101UP") (at 113.03 113.03 270) (unit 1)
+    (in_bom yes) (on_board yes) (dnp no) (fields_autoplaced)
+    (property "Reference" "C2" (at 115.57 110.0582 90)
+      (effects (font (size 1.27 1.27)) (justify left))
+    )
+    (property "Value" "100uF" (at 115.57 112.5982 90)
+      (effects (font (size 1.27 1.27)) (justify left))
+    )
+    (property "Footprint" "Sega GameGear Audio Board Original:C63D" (at 109.22 106.68 0)
+      (effects (font (size 1.27 1.27)) (justify left top) hide)
+    )
+    (property "Datasheet" "http://industrial.panasonic.com/cdbs/www-data/pdf/RDE0000/RDE0000C1259.pdf" (at 105.41 76.2 0)
+      (effects (font (size 1.27 1.27)) (justify left top) hide)
+    )
+    (property "Height" "7.8" (at -283.16 121.92 0)
+      (effects (font (size 1.27 1.27)) (justify left top) hide)
+    )
+    (property "Manufacturer_Name" "Panasonic" (at -583.16 121.92 0)
+      (effects (font (size 1.27 1.27)) (justify left top) hide)
+    )
+    (property "Manufacturer_Part_Number" "EEEFN1E101UP" (at 115.57 115.1382 90)
+      (effects (font (size 1.27 1.27)) (justify left))
+    )
+    (pin "1")
+    (pin "2")
+    (instances
+      (project "sega-gamegear-audio-original"
+        (path "/bc4894cb-9ef9-4d80-9ba0-901cc46c914e"
+          (reference "C2") (unit 1)
+        )
+      )

Commit message: slightly better potentiometer 3d file
Connections:
- net GND: now also VR1.1; no longer VR1.5
- net at IC1.6 (+I2): now also VR1.2; no longer VR1.4
- net at IC1.7 (+I1): now also VR1.3; no longer VR1.2
- net at R1.2: now also VR1.4; no longer VR1.1
- net at R2.2: now also VR1.5; no longer VR1.3
Changed lines of the file:
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@@
-    )
-  )
-  (symbol (lib_id "power:GND") (at 171.45 66.04 0) (unit 1)
-    (in_bom yes) (on_board yes) (dnp no)
-    (property "Reference" "#PWR011" (at 171.45 72.39 0)
-      (effects (font (size 1.27 1.27)) hide)
-    )
-    (property "Value" "GND" (at 171.45 69.85 0)
-      (effects (font (size 1.27 1.27)))
-    )
-    (property "Footprint" "" (at 171.45 66.04 0)
-      (effects (font (size 1.27 1.27)) hide)
-    )
-    (property "Datasheet" "" (at 171.45 66.04 0)
-      (effects (font (size 1.27 1.27)) hide)
-    )
-    (pin "1")
-    (instances
-      (project "sega-gamegear-audio-original"
-        (path "/bc4894cb-9ef9-4d80-9ba0-901cc46c914e"
-          (reference "#PWR011") (unit 1)
-        )
-      )
     )
   )
@@
         )
       )
+    )
+  )
+  (symbol (lib_id "power:GND") (at 171.45 66.04 0) (unit 1)
+    (in_bom yes) (on_board yes) (dnp no)
+    (property "Reference" "#PWR011" (at 171.45 72.39 0)
+      (effects (font (size 1.27 1.27)) hide)
+    )
+    (property "Value" "GND" (at 171.45 69.85 0)
+      (effects (font (size 1.27 1.27)))
+    )
+    (property "Footprint" "" (at 171.45 66.04 0)
+      (effects (font (size 1.27 1.27)) hide)
+    )
+    (property "Datasheet" "" (at 171.45 66.04 0)
+      (effects (font (size 1.27 1.27)) hide)
+    )
+    (pin "1")
+    (instances
+      (project "sega-gamegear-audio-original"
+        (path "/bc4894cb-9ef9-4d80-9ba0-901cc46c914e"
+          (reference "#PWR011") (unit 1)
+        )
+      )

Commit message: trace sizing
Parts:
- renumbered CN2 to CN1, CN1 to CN2
Changed lines of the file:
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@@
   (symbol (lib_id "292161-6:292161-6") (at 26.67 91.44 0) (unit 1)
     (in_bom yes) (on_board yes) (dnp no)
-    (property "Reference" "CN2" (at 33.02 81.28 0)
+    (property "Reference" "CN1" (at 33.02 81.28 0)
       (effects (font (size 1.27 1.27)) (justify left))
     )
@@
       (project "sega-gamegear-audio-original"
         (path "/bc4894cb-9ef9-4d80-9ba0-901cc46c914e"
-          (reference "CN2") (unit 1)
+          (reference "CN1") (unit 1)
         )
       )
@@
   (symbol (lib_id "292161-2:292161-2") (at 243.84 125.73 0) (unit 1)
     (in_bom yes) (on_board yes) (dnp no) (fields_autoplaced)
-    (property "Reference" "CN1" (at 247.65 121.92 0)
+    (property "Reference" "CN2" (at 247.65 121.92 0)
       (effects (font (size 1.27 1.27)) (justify left))
     )
@@
       (project "sega-gamegear-audio-original"
         (path "/bc4894cb-9ef9-4d80-9ba0-901cc46c914e"
-          (reference "CN1") (unit 1)
-        )
-      )
+          (reference "CN2") (unit 1)
+        )
+      )

Commit message: add production files
Parts:
- C1, C2: LCSC Part (none) -> C494824
- C3: LCSC Part (none) -> C178586
- C4, C6, C8: LCSC Part (none) -> C3011705
- C5, C7: LCSC Part (none) -> C336261
Changed lines of the file:
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@@
       (effects (font (size 1.27 1.27)) (justify right))
+    )
+    (property "LCSC Part" "C3011705" (at 182.88 85.09 0)
+      (effects (font (size 1.27 1.27)) hide)
     )
     (pin "1")
@@
       (effects (font (size 1.27 1.27)))
     )
+    (property "LCSC Part" "C336261" (at 161.29 83.82 0)
+      (effects (font (size 1.27 1.27)) hide)
+    )
     (pin "1")
     (pin "2")
@@
       (effects (font (size 1.27 1.27)) (justify right))
     )
+    (property "LCSC Part" "C3011705" (at 215.9 62.23 0)
+      (effects (font (size 1.27 1.27)) hide)
+    )
     (pin "1")
     (pin "2")
@@
     (property "Manufacturer_Part_Number" "GRM188R72A104KA35J" (at 175.26 113.03 90)
       (effects (font (size 1.27 1.27)) (justify right))
+    )
+    (property "LCSC Part" "C3011705" (at 182.88 110.49 0)
+      (effects (font (size 1.27 1.27)) hide)
     )
     (pin "1")
@@
   )
   (symbol (lib_id "EEEFT0J331AP:EEEFT0J331AP") (at 149.86 62.23 270) (unit 1)
-    (in_bom yes) (on_board yes) (dnp no) (fields_autoplaced)
+    (in_bom yes) (on_board yes) (dnp no)
     (property "Reference" "C3" (at 152.4 59.2582 90)
       (effects (font (size 1.27 1.27)) (justify left))
@@
       (effects (font (size 1.27 1.27)) (justify left))
     )
+    (property "LCSC Part" "C178586" (at 146.05 62.23 0)
+      (effects (font (size 1.27 1.27)) hide)
+    )
     (pin "1")
     (pin "2")
@@
       (effects (font (size 1.27 1.27)) (justify left))
     )
+    (property "LCSC Part" "C494824" (at 113.03 90.17 0)
+      (effects (font (size 1.27 1.27)) hide)
+    )
     (pin "1")
     (pin "2")
@@
       (effects (font (size 1.27 1.27)))
     )
+    (property "LCSC Part" "C336261" (at 161.29 109.22 0)
+      (effects (font (size 1.27 1.27)) hide)
+    )
     (pin "1")
     (pin "2")
@@
       (effects (font (size 1.27 1.27)) (justify left))
     )
-    (pin "1")
+    (property "LCSC Part" "C494824" (at 113.03 113.03 0)
+      (effects (font (size 1.27 1.27)) hide)
+    )
+    (pin "1")

Commit message: update production files
Parts:
- CN1: LCSC Part (none) -> C499123
- CN2: LCSC Part (none) -> C86484
- IC1: LCSC Part (none) -> C668663
Changed lines of the file:
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@@
       (effects (font (size 1.27 1.27)) hide)
+    )
+    (property "LCSC Part" "C668663" (at 142.24 93.98 0)
+      (effects (font (size 1.27 1.27)))
     )
     (pin "4")
@@
       (effects (font (size 1.27 1.27)) hide)
     )
+    (property "LCSC Part" "C499123" (at 26.67 101.6 0)
+      (effects (font (size 1.27 1.27)) hide)
+    )
     (pin "1")
     (pin "2")
@@
       (effects (font (size 1.27 1.27)) (justify left))
     )
-    (pin "1")
+    (property "LCSC Part" "C86484" (at 243.84 134.62 0)
+      (effects (font (size 1.27 1.27)) hide)
+    )
+    (pin "1")
